File: ESP32-Sprinkler-System/ESP32-Sprinkler-System.kicad_pcb (KiCad board)
At the start: 4 copper layers, 58 parts, among them J101 12V, J102 DHT, J103 NEOPIXEL, J104 LCD, J105 BME280, J201 TBL004-508-02BE-2GY, J202 TBL004-508-02BE-2GY, J203 TBL004-508-02BE-2GY, J204 TBL004-508-02BE-2GY, Q201 IRFZ24NPBF, Q202 IRFZ24NPBF, Q203 IRFZ24NPBF, Q204 IRFZ24NPBF, U101 V7805-500, U102 ESP32-DEVKITC-32D, U201 MC33152PG, U202 MC33152PG

Commit message: Objs sorted like the schematic
Parts:
- moved J103 142.0 mm to (11.0, 186.8)
- moved J102 136.1 mm to (28.8, 183.0)
- moved J104 135.4 mm to (44.0, 179.2)
- moved S101 132.5 mm to (84.7, 188.1)
- moved J105 124.6 mm to (59.3, 176.6)
- moved J201 118.3 mm to (273.3, 29.4), turned to -90 degrees
- moved D208 114.6 mm to (254.9, 141.1), turned to -90 degrees
- moved J204 110.0 mm to (272.3, 143.7), turned to -90 degrees
- moved J203 107.2 mm to (272.3, 100.5), turned to -90 degrees
- moved R201 101.9 mm to (247.2, 28.0), turned to -90 degrees
- moved R217 99.1 mm to (154.5, 146.2)
- moved D206 98.2 mm to (254.9, 97.9), turned to -90 degrees
- moved R216 93.5 mm to (249.8, 144.9), turned to -90 degrees
- moved D204 91.0 mm to (254.9, 67.4), turned to -90 degrees
- moved D201 90.7 mm to (249.8, 22.9)
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
Commit message: compact formation
Parts:
- moved C206 114.8 mm to (158.0, 120.1)
- moved C202 108.0 mm to (164.3, 82.7)
- moved C203 106.2 mm to (158.0, 83.2)
- moved C101 101.4 mm to (136.8, 79.6)
- moved C205 100.8 mm to (164.3, 118.3)
- moved J101 90.0 mm to (116.1, 64.9)
- moved C102 89.5 mm to (138.0, 70.6)
- moved D201 88.4 mm to (171.9, 64.9), turned to 90 degrees
- moved J201 86.3 mm to (195.8, 67.6)
- moved U101 84.9 mm to (142.4, 71.8)
- moved D202 82.2 mm to (180.8, 63.8)
- moved J204 79.8 mm to (195.8, 120.8)
- moved R201 79.4 mm to (177.0, 65.0)
- moved J102 79.2 mm to (98.3, 144.9)
- moved J103 79.2 mm to (80.5, 148.8)
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
Commit message: good layout.
Parts:
- moved J201 125.1 mm to (70.7, 66.1)
- moved J202 125.1 mm to (70.7, 83.9)
- moved J203 125.1 mm to (70.7, 101.8)
- moved J204 125.1 mm to (70.7, 119.5)
- moved D204 105.0 mm to (75.8, 82.6)
- moved D206 105.0 mm to (75.8, 100.4)
- moved D208 105.0 mm to (75.8, 118.2)
- moved D202 105.0 mm to (75.8, 64.9)
- moved R206 97.4 mm to (79.6, 83.9)
- moved R211 97.4 mm to (79.6, 101.7)
- moved R216 97.4 mm to (79.6, 119.5)
- moved R201 97.4 mm to (79.6, 66.1)
- moved Q204 88.2 mm to (84.4, 130.9), turned to 90 degrees
- moved Q201 87.9 mm to (84.7, 77.6), turned to 90 degrees
- moved Q203 87.9 mm to (84.7, 113.1), turned to 90 degrees
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Routing:
- added copper zone on B.Cu, net GND
Other:
- board outline added: 207 x 158.8 mm
- copper layers 4 -> 2

Commit message: going to edit tracks
Routing:
- net 12V: track 0.00 -> 241.9 mm
- net Net-(R218-Pad1): track 0.00 -> 37.1 mm
- net 5V: track 0.00 -> 30.7 mm
- net Net-(R202-Pad1): track 0.00 -> 26.8 mm
- net Net-(D204-Pad2): track 0.00 -> 26.0 mm
- net Net-(D202-Pad2): track 0.00 -> 26.0 mm
- net Net-(D206-Pad2): track 0.00 -> 25.9 mm
- net Net-(D208-Pad2): track 0.00 -> 25.6 mm
- net Net-(R208-Pad1): track 0.00 -> 15.9 mm
- net Net-(R207-Pad2): track 0.00 -> 14.7 mm
- net Net-(R217-Pad2): track 0.00 -> 14.1 mm
- net Net-(R212-Pad1): track 0.00 -> 13.0 mm
- net Net-(R214-Pad2): track 0.00 -> 9.19 mm
- net Net-(R204-Pad2): track 0.00 -> 8.00 mm
