File: ESP32-Sprinkler-System/ESP32-Sprinkler-System-rounded.kicad_pcb (KiCad board)
At the start: 2 copper layers, 135 x 87 mm, 62 parts, among them J101 12V, J102 DHT, J103 NEOPIXEL, J104 LCD, J105 BME280, J201 TBL004-508-02BE-2GY, J202 TBL004-508-02BE-2GY, J203 TBL004-508-02BE-2GY, J204 TBL004-508-02BE-2GY, Q201 IRFZ24NPBF, Q202 IRFZ24NPBF, Q203 IRFZ24NPBF, Q204 IRFZ24NPBF, U101 V7805-500, U102 ESP32-DEVKITC-32D, U201 MC33152PG, U202 MC33152PG

Commit message: Updated PCB
Other:
- board text added: "Sprinkler System"
- board text removed: "ESP32 Wireless Sprinkler System"
Changed lines of the file:
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@@
       (net 55 "unconnected-(U102-Pad38)") (pinfunction "CLK") (pintype "input"))
     (model "${KIPRJMOD}/Snap EDA/ESP32-DEVKITC-32D/ESP32-DEVKITC-32D.step"
-      (offset (xyz 0 -3.08 10.45))
+      (offset (xyz 0 -3.08 3.5))
       (scale (xyz 1 1 1))
       (rotate (xyz -90 0 0))
-    )
-    (model "${KICAD6_3DMODEL_DIR}/Connector_PinSocket_2.54mm.3dshapes/PinSocket_1x19_P2.54mm_Vertical.step"
-      (offset (xyz 12.7 19.8 0))
-      (scale (xyz 1 1 1))
-      (rotate (xyz 0 0 0))
-    )
-    (model "${KICAD6_3DMODEL_DIR}/Connector_PinSocket_2.54mm.3dshapes/PinSocket_1x19_P2.54mm_Vertical.step"
-      (offset (xyz -12.7 19.8 0))
-      (scale (xyz 1 1 1))
-      (rotate (xyz 0 0 0))
     )
   )
@@
     (effects (font (size 1 1) (thickness 0.15)))
   )
-  (gr_text "ESP32 Wireless Sprinkler System" (at 162 58) (layer "F.SilkS")
+  (gr_text "Sprinkler System" (at 174.244 59.944) (layer "F.SilkS")
     (effects (font (size 1.5 1.5) (thickness 0.3)))
   )
@@
     (effects (font (size 1 1) (thickness 0.15)))
   )
-  (gr_text "https://github.com/mrangen/ESP32-Sprinkler-System" (at 164 61) (layer "F.SilkS")
+  (gr_text "https://github.com/mrangen/ESP32-Sprinkler-System" (at 162.306 56.642) (layer "F.SilkS")
     (effects (font (size 1 1) (thickness 0.15)))
   )
@@
     (effects (font (size 1.5 1) (thickness 0.15)) (justify left))
   )
-  (gr_text "J&R Creative Technologies Inc." (at 106 58.166) (layer "F.SilkS")
+  (gr_text "J&R Creative Technologies Inc." (at 94.234 58.166) (layer "F.SilkS")
     (effects (font (size 2 2) (thickness 0.25)))
   )
@@
   )
   (dimension (type aligned) (layer "Dwgs.User")
-    (pts (xy 62 57) (xy 62 136))
-    (height 9)
-    (gr_text "79.0000 mm" (at 51.85 96.5 90) (layer "Dwgs.User")
-      (effects (font (size 1 1) (thickness 0.15)))
-    )
-    (format (units 3) (units_format 1) (precision 4))
-    (style (thickness 0.15) (arrow_length 1.27) (text_position_mode 0) (extension_height 0.58642) (extension_offset 0.5) keep_text_aligned)
-  )
-  (dimension (type aligned) (layer "Dwgs.User")
     (pts (xy 355.28 36.6) (xy 300.78 36.6))
     (height 5.49)
@@
       (effects (font (size 1 1) (thickness 0.15)))
     )
-    (format (units 3) (units_format 1) (precision 4))
-    (style (thickness 0.15) (arrow_length 1.27) (text_position_mode 0) (extension_height 0.58642) (extension_offset 0.5) keep_text_aligned)
-  )
-  (dimension (type aligned) (layer "Dwgs.User")
-    (pts (xy 189 57) (xy 62 57))
-    (height 9.999999)
-    (gr_text "127.0000 mm" (at 125.5 45.850001) (layer "Dwgs.User")
-      (effects (font (size 1 1) (thickness 0.15)))
-    )
